Commit message: Change color of meshes, scripts to yaw and custom world

File: src/LandMark_description/urdf/LandMark1.xacro (robot description, xacro)
@@ -23,3 +23,8 @@
   </collision>
 </link>
+<link name="world"/>
+<joint name="base_link_joint" type="fixed">
+  <parent link="world"/>
+  <child link="base_link"/>
+</joint>
 </robot>

File: src/LandMark_description/urdf/LandMark2.xacro (robot description, xacro)
@@ -13,5 +13,5 @@
     <origin xyz="0 0 0.57" rpy="0 0 0"/>
     <geometry>
-      <mesh filename="package://LandMark2_description/meshes/LandMark2.dae"/>
+      <mesh filename="package://LandMark_description/meshes/LandMark2.dae"/>
     </geometry>
   </visual>
@@ -19,5 +19,5 @@
     <origin xyz="0 0 0" rpy="0 0 0"/>
     <geometry>
-      <mesh filename="package://LandMark2_description/meshes/LandMark2.dae"/>
+      <mesh filename="package://LandMark_description/meshes/LandMark2.dae"/>
     </geometry>
   </collision>

Commit message: OK but angle in landmarks

File: src/LandMark_description/urdf/LandMark1.xacro (robot description, xacro)
@@ -11,5 +11,5 @@
   </inertial>
   <visual>
-    <origin xyz="0 0 0.57" rpy="0 0 0"/>
+    <origin xyz="0 0 0.57" rpy="0 0 0.785"/>
     <geometry>
       <mesh filename="package://LandMark_description/meshes/LandMark1.dae"/>
@@ -23,8 +23,3 @@
   </collision>
 </link>
-<link name="world"/>
-<joint name="base_link_joint" type="fixed">
-  <parent link="world"/>
-  <child link="base_link"/>
-</joint>
 </robot>
