Commit message: change position of camera

File: src/ERC22_URDF_description/urdf/ERC22_URDF.xacro (robot description, xacro)
@@ -285,4 +285,5 @@
   </inertial>
 </link>
+<!--
 <link name="camera_link_right">
   <collision>
@@ -304,5 +305,5 @@
     <inertia ixx="1e-6" ixy="0" ixz="0" iyy="1e-6" iyz="0" izz="1e-6" />
   </inertial>
-</link>
+</link> -->
 <joint name="S_LF" type="continuous">
   <origin xyz="0.391355 -0.383158 0.356565" rpy="0 0 0"/>
@@ -379,13 +380,13 @@
 <joint name="camera_joint_left" type="fixed">
   <axis xyz="0 1 0" />
-  <origin xyz="0.285 0.23 0.58" rpy="0 0 0.785"/>
+  <origin xyz="0.285 0 0.58" rpy="0 0 0"/>
   <parent link="base_link"/>
   <child link="camera_link_left"/>
 </joint>
-<joint name="camera_joint_right" type="fixed">
+<!-- <joint name="camera_joint_right" type="fixed">
   <axis xyz="0 1 0" />
   <origin xyz="0.285 -0.23 0.58" rpy="0 0 -0.785"/>
   <parent link="base_link"/>
   <child link="camera_link_right"/>
-</joint>
+</joint> -->
 </robot>
